File: kicad/V3.kicad_pcb (KiCad board)
At the start: 2 copper layers, 175.6 x 118.3 mm, 51 parts, among them SW1 Slide_Switch_SPDT_P3mm_10x5x1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

Commit message: positioning
Parts:
- moved CH16 0.64 mm to (109.5, 101.0)
- moved D16 0.64 mm to (103.8, 110.4)
Routing:
- net /Row3: track 309.2 -> 310.1 mm
Changed lines of the file:
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@@
 	(footprint "Diode_THT:D_DO-35_SOD27_P7.62mm_Horizontal"
 		(layer "F.Cu")
-		(at 104.416033 110.404027 5)
+		(at 103.772593 110.404027 5)
 		(descr "Diode, DO-35_SOD27 series, Axial, Horizontal, pin pitch=7.62mm, , length*diameter=4*2mm^2, , http://www.diodes.com/_files/packages/DO-35.pdf")
 		(tags "Diode DO-35_SOD27 series Axial Horizontal pin pitch 7.62mm  length 4mm diameter 2mm")
@@
 		)
 		(fp_arc
-			(start -2.461268 -0.627505)
+			(start -2.461268 -0.627506)
 			(mid -1.558484 -2.005674)
 			(end 0 -2.540001)
@@
 		(fp_line
 			(start -8.89 1.27)
-			(end -8.889998 3.81)
+			(end -8.889997 3.81)
 			(stroke
 				(width 0.12)
@@
 		)
 		(fp_line
-			(start -8.889998 3.81)
+			(start -8.889997 3.81)
 			(end -6.35 3.81)
 			(stroke
@@
 		)
 		(fp_arc
-			(start -2.461268 -0.627505)
+			(start -2.461268 -0.627506)
 			(mid -1.558484 -2.005674)
 			(end 0 -2.540001)
@@
 		(fp_line
 			(start -8.89 1.27)
-			(end -8.889998 3.81)
+			(end -8.889997 3.81)
 			(stroke
 				(width 0.12)
@@
 		)
 		(fp_line
-			(start -8.889998 3.81)
+			(start -8.889997 3.81)
 			(end -6.35 3.81)
 			(stroke
@@
 		)
 		(fp_arc
-			(start -2.461268 -0.627505)
+			(start -2.461268 -0.627506)
 			(mid -1.558484 -2.005674)
 			(end 0 -2.540001)
@@
 		(fp_line
 			(start -8.89 1.27)
-			(end -8.889998 3.81)
+			(end -8.889997 3.81)
 			(stroke
 				(width 0.12)
@@
 		)
 		(fp_line
-			(start -8.889998 3.81)
+			(start -8.889997 3.81)
 			(end -6.35 3.81)
 			(stroke
@@
 		)
 		(fp_arc
-			(start -2.461268 -0.627505)
+			(start -2.461268 -0.627506)
 			(mid -1.558484 -2.005674)
 			(end 0 -2.540001)
@@
 		(fp_line
 			(start -8.89 1.27)
-			(end -8.889998 3.81)
+			(end -8.889997 3.81)
 			(stroke
 				(width 0.12)
@@
 		)
 		(fp_line
-			(start -8.889998 3.81)
+			(start -8.889997 3.81)
 			(end -6.35 3.81)
 			(stroke
@@
 		)
 		(fp_arc
-			(start -2.461268 -0.627505)
+			(start -2.461268 -0.627506)
 			(mid -1.558484 -2.005674)
 			(end 0 -2.540001)
@@
 		(fp_line
 			(start -8.89 1.27)
-			(end -8.889998 3.81)
+			(end -8.889997 3.81)
 			(stroke
 				(width 0.12)
@@
 		)
 		(fp_line
-			(start -8.889998 3.81)
+			(start -8.889997 3.81)
 			(end -6.35 3.81)
 			(stroke
@@
 	(footprint "Library:Kailh_socket_MX_reversible"
 		(layer "F.Cu")
-		(at 110.160317 100.977509 5)
+		(at 109.516877 100.977509 5)
 		(descr "MX-style keyswitch with reversible Kailh socket mount")
 		(tags "MX,cherry,gateron,kailh,pg1511,socket")
@@
 		)
 		(fp_arc
-			(start -2.461268 -0.627505)
+			(start -2.461268 -0.627506)
 			(mid -1.558484 -2.005674)
 			(end 0 -2.540001)
@@
 		(fp_line
 			(start -8.89 1.27)
-			(end -8.889998 3.81)
+			(end -8.889997 3.81)
 			(stroke
 				(width 0.12)
@@
 		)
 		(fp_line
-			(start -8.889998 3.81)
+			(start -8.889997 3.81)
 			(end -6.35 3.81)
 			(stroke
@@
 		)
 		(fp_arc
-			(start -2.461268 -0.627505)
+			(start -2.461268 -0.627506)
 			(mid -1.558484 -2.005674)
 			(end 0 -2.540001)
@@
 		(fp_line
 			(start -8.89 1.27)
-			(end -8.889998 3.81)
+			(end -8.889997 3.81)
 			(stroke
 				(width 0.12)
@@
 		)
 		(fp_line
-			(start -8.889998 3.81)
+			(start -8.889997 3.81)
 			(end -6.35 3.81)
 			(stroke
@@
 	)
 	(segment
-		(start 102.85046 104.166741)
-		(end 102.651222 101.88944)
+		(start 102.20702 104.166741)
+		(end 102.007782 101.88944)
 		(width 0.2)
 		(layer "F.Cu")
@@
 	)
 	(segment
-		(start 102.85046 104.166741)
-		(end 109.729736 109.939138)
+		(start 102.20702 104.166741)
+		(end 109.086296 109.939138)
 		(width 0.2)
 		(layer "F.Cu")
@@
 	)
 	(segment
-		(start 109.729736 109.939138)
-		(end 112.007037 109.7399)
+		(start 109.086296 109.939138)
+		(end 111.363597 109.7399)
 		(width 0.2)
 		(layer "F.Cu")
@@
 	)
 	(segment
-		(start 102.651222 101.88944)
-		(end 102.376051 101.658544)
+		(start 102.007782 101.88944)
+		(end 101.732611 101.658544)
 		(width 0.2)
 		(layer "F.Cu")
@@
 	)
 	(via
-		(at 102.376051 101.658544)
+		(at 101.732611 101.658544)
 		(size 0.6)
 		(drill 0.3)
@@
 	)
 	(segment
-		(start 102.407709 99.106072)
-		(end 102.606947 101.383373)
+		(start 101.764269 99.106072)
+		(end 101.963507 101.383373)
 		(width 0.2)
 		(layer "B.Cu")
@@
 	)
 	(segment
-		(start 102.606947 101.383373)
-		(end 102.376051 101.658544)
+		(start 101.963507 101.383373)
+		(end 101.732611 101.658544)
 		(width 0.2)
 		(layer "B.Cu")
@@
 	)
 	(segment
+		(start 102.755716 91.426518)
+		(end 102.564091 91.426518)
+		(width 0.2)
+		(layer "F.Cu")
+		(net 33)
+	)
+	(segment
+		(start 102.564091 91.426518)
+		(end 99.756047 94.234562)
+		(width 0.2)
+		(layer "F.Cu")
+		(net 33)
+	)
+	(segment
 		(start 194.802 55.6007)
 		(end 194.802 71.962)
@@
 	)
 	(segment
-		(start 101.607989 108.047798)
-		(end 104.416033 110.404027)
+		(start 100.964549 108.047798)
+		(end 103.772593 110.404027)
 		(width 0.2)
 		(layer "F.Cu")
@@
 	)
 	(segment
-		(start 102.755716 91.426518)
-		(end 100.399487 94.234562)
-		(width 0.2)
-		(layer "F.Cu")
-		(net 33)
-	)
-	(segment
 		(start 164.490795 47.009205)
 		(end 164.778591 47.297)
@@
 	)
 	(segment
-		(start 100.399487 94.234562)
-		(end 101.607989 108.047798)
+		(start 99.756047 94.234562)
+		(end 100.964549 108.047798)
 		(width 0.2)
 		(layer "F.Cu")
@@
 	)
 	(segment
-		(start 116.869133 105.489968)
-		(end 116.327373 99.297622)
+		(start 116.225693 105.489968)
+		(end 115.683933 99.297622)
 		(width 0.2)
 		(layer "F.Cu")
@@
 	)
 	(segment
-		(start 116.327373 99.297622)
-		(end 116.182204 99.175811)
+		(start 115.683933 99.297622)
+		(end 115.538764 99.175811)
 		(width 0.2)
 		(layer "F.Cu")
@@
 	)
 	(via
-		(at 116.182204 99.175811)
+		(at 115.538764 99.175811)
 		(size 0.6)
 		(drill 0.3)
@@
 	)
 	(segment
-		(start 113.978349 93.685999)
-		(end 98.688752 95.023666)
-		(width 0.2)
-		(layer "B.Cu")
-		(net 35)
-	)
-	(segment
 		(start 187.471 89.679)
 		(end 173.421 89.679)
@@
 	)
 	(segment
-		(start 116.304015 99.030642)
-		(end 116.182204 99.175811)
+		(start 115.660575 99.030642)
+		(end 115.538764 99.175811)
 		(width 0.2)
 		(layer "B.Cu")
@@
 	)
 	(segment
+		(start 98.688752 95.023666)
+		(end 99.867954 93.844464)
+		(width 0.2)
+		(layer "B.Cu")
+		(net 35)
+	)
+	(segment
 		(start 159.377709 85.658)
 		(end 153.35 85.658)
@@
 	)
 	(segment
-		(start 115.98363 95.36863)
-		(end 116.304015 99.030642)
+		(start 115.34019 95.36863)
+		(end 115.660575 99.030642)
 		(width 0.2)
 		(layer "B.Cu")
@@
 	)
 	(segment
-		(start 153.35 89.334)
-		(end 153.216 89.468)
+		(start 115.34019 92.324158)
+		(end 118.317348 89.347)
 		(width 0.2)
 		(layer "B.Cu")
@@
 	)
 	(segment
-		(start 115.98363 95.36863)
-		(end 113.978349 93.685999)
+		(start 153.35 89.334)
+		(end 153.216 89.468)
 		(width 0.2)
 		(layer "B.Cu")
@@
 	)
 	(segment
+		(start 99.867954 93.844464)
+		(end 113.816024 93.844464)
+		(width 0.2)
+		(layer "B.Cu")
+		(net 35)
+	)
+	(segment
+		(start 115.34019 95.36863)
+		(end 115.34019 92.324158)
+		(width 0.2)
+		(layer "B.Cu")
+		(net 35)
+	)
+	(segment
 		(start 132.449 90.509)
 		(end 134.3 88.658)
@@
 	)
 	(segment
-		(start 113.978349 93.685999)
-		(end 118.317348 89.347)
+		(start 113.816024 93.844464)
+		(end 115.34019 95.36863)
 		(width 0.2)
 		(layer "B.Cu")

Commit message: filled area
Routing:
- added copper zone on F.Cu, net Earth
Changed lines of the file:
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@@
 	)
 	(paper "A4")
+	(title_block
+		(title "Wing23")
+		(rev "3")
+	)
 	(layers
 		(0 "F.Cu" signal)
@@
 		(fp_line
 			(start -8.89 1.27)
-			(end -8.889997 3.81)
+			(end -8.889996 3.81)
 			(stroke
 				(width 0.12)
@@
 		)
 		(fp_line
-			(start -8.889997 3.81)
+			(start -8.889996 3.81)
 			(end -6.35 3.81)
 			(stroke
@@
 		(fp_line
 			(start -8.89 1.27)
-			(end -8.889997 3.81)
+			(end -8.889996 3.81)
 			(stroke
 				(width 0.12)
@@
 		)
 		(fp_line
-			(start -8.889997 3.81)
+			(start -8.889996 3.81)
 			(end -6.35 3.81)
 			(stroke
@@
 		(fp_line
 			(start -8.89 1.27)
-			(end -8.889997 3.81)
+			(end -8.889996 3.81)
 			(stroke
 				(width 0.12)
@@
 		)
 		(fp_line
-			(start -8.889997 3.81)
+			(start -8.889996 3.81)
 			(end -6.35 3.81)
 			(stroke
@@
 		(fp_line
 			(start -8.89 1.27)
-			(end -8.889997 3.81)
+			(end -8.889996 3.81)
 			(stroke
 				(width 0.12)
@@
 		)
 		(fp_line
-			(start -8.889997 3.81)
+			(start -8.889996 3.81)
 			(end -6.35 3.81)
 			(stroke
@@
 		(fp_line
 			(start -8.89 1.27)
-			(end -8.889997 3.81)
+			(end -8.889996 3.81)
 			(stroke
 				(width 0.12)
@@
 		)
 		(fp_line
-			(start -8.889997 3.81)
+			(start -8.889996 3.81)
 			(end -6.35 3.81)
 			(stroke
@@
 		(fp_line
 			(start -8.89 1.27)
-			(end -8.889997 3.81)
+			(end -8.889996 3.81)
 			(stroke
 				(width 0.12)
@@
 		)
 		(fp_line
-			(start -8.889997 3.81)
+			(start -8.889996 3.81)
 			(end -6.35 3.81)
 			(stroke
@@
 		(fp_line
 			(start -8.89 1.27)
-			(end -8.889997 3.81)
+			(end -8.889996 3.81)
 			(stroke
 				(width 0.12)
@@
 		)
 		(fp_line
-			(start -8.889997 3.81)
+			(start -8.889996 3.81)
 			(end -6.35 3.81)
 			(stroke
@@
 		(layer "Edge.Cuts")
 	)
+	(dimension
+		(type orthogonal)
+		(layer "F.Cu")
+		(pts
+			(xy 190.24 86.673) (xy 190.24 72.703)
+		)
+		(height 12.76)
+		(orientation 1)
+		(format
+			(prefix "")
+			(suffix "")
+			(units 3)
+			(units_format 0)
+			(precision 4)
+			(suppress_zeroes yes)
+		)
+		(style
+			(thickness 0.2)
+			(arrow_length 1.27)
+			(text_position_mode 0)
+			(arrow_direction outward)
+			(extension_height 0.58642)
+			(extension_offset 0.5)
+			(keep_text_aligned yes)
+		)
+		(gr_text "13.97"
+			(at 201.2 79.688 90)
+			(layer "F.Cu")
+			(effects
+				(font
+					(size 1.5 1.5)
+					(thickness 0.3)
+				)
+			)
+		)
+	)
 	(segment
 		(start 99.330589 63.934422)
@@
 	)
 	(segment
-		(start 227.5 96.150057)
+		(start 227.5 80)
 		(end 227.5 79)
 		(width 0.2)
@@
 	)
 	(segment
-		(start 219.719 70.781)
-		(end 225.556049 70.781)
-		(width 0.2)
-		(layer "F.Cu")
-		(net 8)
-	)
-	(segment
-		(start 227.5 79)
-		(end 227.5 68.837049)
+		(start 229.5 81)
+		(end 227.5 79)
 		(width 0.2)
 		(layer "F.Cu")
@@
 	)
 	(segment
-		(start 229.5 81)
-		(end 227.5 79)
+		(start 226.719 70.781)
+		(end 227.5 71.562)
 		(width 0.2)
 		(layer "F.Cu")
@@
 	)
 	(segment
-		(start 227.5 97.5)
-		(end 227.5 96.849943)
+		(start 228.301 66.341)
+		(end 228.301 69.199)
 		(width 0.2)
 		(layer "F.Cu")
@@
 	)
 	(segment
-		(start 228.301 68.036049)
+		(start 227 65.04)
 		(end 228.301 66.341)
 		(width 0.2)
@@
 	)
 	(segment
-		(start 227.5 68.837049)
-		(end 228.301 68.036049)
+		(start 227.5 71.562)
+		(end 227.5 80)
 		(width 0.2)
 		(layer "F.Cu")
@@
 	)
 	(segment
-		(start 229.5 86)
-		(end 229.5 81)
+		(start 227.5 97.5)
+		(end 227.5 96.849943)
 		(width 0.2)
 		(layer "F.Cu")
@@
 	)
 	(segment
-		(start 228.301 66.341)
-		(end 227 65.04)
+		(start 219.719 70.781)
+		(end 203.5 87)
+		(width 0.2)
+		(layer "F.Cu")
+		(net 8)
+	)
+	(segment
+		(start 229.5 86)
+		(end 229.5 81)
 		(width 0.2)
 		(layer "F.Cu")
@@
 	)
 	(segment
-		(start 225.556049 70.781)
-		(end 227.5 68.837049)
+		(start 226.719 70.781)
+		(end 219.719 70.781)
 		(width 0.2)
 		(layer "F.Cu")
@@
 	)
 	(segment
-		(start 203.5 87)
-		(end 219.719 70.781)
+		(start 228.301 69.199)
+		(end 226.719 70.781)
+		(width 0.2)
+		(layer "F.Cu")
+		(net 8)
+	)
+	(segment
+		(start 227.5 96.150057)
+		(end 227.5 80)
 		(width 0.2)
 		(layer "F.Cu")
@@
 		(net 55)
 	)
+	(zone
+		(net 11)
+		(net_name "Earth")
+		(layer "F.Cu")
+		(hatch edge 0.5)
+		(connect_pads
+			(clearance 0.5)
+		)
+		(min_thickness 0.25)
+		(filled_areas_thickness no)
+		(fill
+			(thermal_gap 0.5)
+			(thermal_bridge_width 0.5)
+		)
+		(polygon
+			(pts
+				(xy 194.5 62) (xy 229.5 62) (xy 229.5 103) (xy 202 130) (xy 192 130) (xy 190 128) (xy 190 109) (xy 194.5 107)
+			)
+		)
+	)
 	(embedded_fonts no)

Commit message: lots of changes
usb module support and more fixed wirign
Connections:
- A1 pad 20: unconnected-(A1-ADC1_CH7/D35-Pad20) -> /USB_rst
- Brd1 pad 2: VCC -> /~3v3
- SW1 pad 3: VCC -> +5V
- U1 pad 2: VCC -> +5V
- U2 pad 1: VCC -> +5V
- U2 pad 4: unconnected-(U2-RST-Pad4) -> /USB_rst
Routing:
- net VCC: track 113.3 -> 0.00 mm
- net +5V: track 0.00 -> 106.4 mm
- net /USB_rst: track 0.00 -> 51.9 mm, vias 0 -> 1
- net /~3v3: track 41.7 -> 36.2 mm
- net /Col1: track 200.2 -> 200.9 mm
- removed copper zone on F.Cu, net Earth
