File: kicad_nrf52840/V3.kicad_pcb (KiCad board)
At the start: 2 copper layers, 46 parts, among them SW1 KS33_SW_HS, SW10 KS33_SW_HS, SW11 KS33_SW_HS, SW12 KS33_SW_HS, SW13 KS33_SW_HS, SW14 KS33_SW_HS, SW15 KS33_SW_HS, SW16 KS33_SW_HS, SW17 KS33_SW_HS, SW18 KS33_SW_HS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

Commit message: routing
Parts:
- SW1, SW10, SW11, SW12, SW13, SW14, SW15, SW16, SW17, SW18, SW19, SW2, SW20, SW21, SW22, SW3, SW4, SW5, SW6, SW7, SW8, SW9: moved to B.Cu
- moved SW22 126.2 mm to (198.5, 136.7), turned to -75 degrees
- moved D22 123.1 mm to (191.2, 142.5), turned to 105 degrees
- moved SW4 115.5 mm to (179.8, 48.5)
- moved U4 102.7 mm to (185.3, 103.5), turned to 0 degrees
- moved SW6 100.6 mm to (141.7, 56.5)
- moved SW10 91.6 mm to (179.8, 67.6)
- moved SW2 87.8 mm to (160.7, 42.5)
- moved SW12 74.6 mm to (141.7, 75.6)
- moved D18 70.3 mm to (91.4, 105.3), turned to -172 degrees
- moved SW16 69.1 mm to (179.8, 86.6)
- moved SW5 67.2 mm to (99.7, 54.1), turned to 8 degrees
- moved SW8 66.6 mm to (160.7, 61.5)
- moved SW1 66.5 mm to (141.7, 37.5)
- moved D7 66.3 mm to (86.1, 67.6), turned to -172 degrees
- moved SW21 66.2 mm to (186.4, 119.5), turned to -55 degrees
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Connections:
- D1 pad 1: /Row4 -> /Row1
- D11 pad 1: Net-(D11-K) -> /Row2
- D12 pad 1: /Row2 -> /Row3
- D13 pad 1: /Row3 -> /Row2
- D17 pad 1: /Row2 -> /Row3
- D19 pad 1: /Row3 -> /Row4
- D2 pad 1: unconnected-(D2-K-Pad1) -> /Row1
- D3 pad 1: unconnected-(D3-K-Pad1) -> /Row1
- D6 pad 1: Net-(D11-K) -> /Row2
- D7 pad 1: /Row2 -> /Row1
- SW1 pad 1: /Col3 -> /Col4
- SW10 pad 1: /Col2 -> /Col6
- SW11 pad 1: /Col6 -> /Col2
- SW12 pad 1: /Col5 -> /Col4
- SW13 pad 1: /Col3 -> /Col1
- SW14 pad 1: /Col4 -> /Col5
- SW15 pad 1: /Col1 -> /Col3
- SW16 pad 1: /Col2 -> /Col6
- SW17 pad 1: /Col6 -> /Col2
- SW18 pad 1: /Col5 -> /Col1
- SW19 pad 1: /Col6 -> /Col3
- SW2 pad 1: /Col3 -> /Col5
- SW3 pad 1: /Col4 -> /Col3
- SW4 pad 1: /Col1 -> /Col6
- SW6 pad 1: /Col5 -> /Col4
- SW7 pad 1: /Col3 -> /Col1
- SW8 pad 1: /Col4 -> /Col5
- SW9 pad 1: /Col1 -> /Col3
- U1 pad 16: unconnected-(U1-3V3-Pad16) -> +3V3
Routing:
- net /Col3: track 0.00 -> 262.1 mm, vias 0 -> 4
- net /Col4: track 0.00 -> 256.7 mm, vias 0 -> 4
- net /Col1: track 0.00 -> 218.8 mm, vias 0 -> 4
- net /Col2: track 0.00 -> 179.5 mm, vias 0 -> 4
- net /Col5: track 0.00 -> 172.7 mm, vias 0 -> 4
- net /Row3: track 0.00 -> 166.2 mm
- net /Col6: track 0.00 -> 164.4 mm, vias 0 -> 4
- net /Row4: track 0.00 -> 156.1 mm
- net /Row1: track 0.00 -> 149.8 mm
- net /Row2: track 0.00 -> 148.1 mm
- net Earth: track 0.00 -> 69.5 mm, vias 0 -> 3
- net +3V3: track 0.00 -> 42.6 mm
- net /SDA: track 0.00 -> 14.7 mm, vias 0 -> 1
- net Net-(D20-A): track 0.00 -> 12.5 mm, vias 0 -> 1
- net Net-(D22-A): track 0.00 -> 12.5 mm, vias 0 -> 1
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
Commit message: full routing
Parts:
- moved SW22 39.3 mm to (159.8, 130.0), turned to -30 degrees
- moved D22 32.7 mm to (158.7, 139.2), turned to 150 degrees
- moved U1 1.27 mm to (198.9, 58.0)
Connections:
- U1 pad 10: unconnected-(U1-P0.11-Pad10) -> /Col1
- U1 pad 26: /Col1 -> unconnected-(U1-P1.02-LF-Pad26)
- U1 pad 27: /Col2 -> unconnected-(U1-P1.07-LF-Pad27)
- U1 pad 9: unconnected-(U1-P1.00-Pad9) -> /Col2
Routing:
- net /Col3: track 262.1 -> 187.1 mm, vias 4 -> 7
- net /Col2: track 179.5 -> 224.9 mm
- net Net-(D2-A): track 12.5 -> 50.3 mm
- net /Row1: track 149.8 -> 179.6 mm
- net Net-(D4-A): track 12.5 -> 34.7 mm, vias 1 -> 0
- net /Col6: track 164.4 -> 144.3 mm, vias 4 -> 6
- net Net-(D1-A): track 12.5 -> 28.1 mm
- net Net-(D8-A): track 12.5 -> 22.5 mm, vias 1 -> 2
- net /Col1: track 218.8 -> 209.2 mm, vias 4 -> 5
- net +3V3: track 42.6 -> 33.2 mm, vias 0 -> 5
- net /Col5: track 172.7 -> 182.1 mm, vias 4 -> 9
- net Net-(D21-A): track 12.5 -> 21.0 mm, vias 1 -> 0
- net Net-(D11-A): track 12.5 -> 20.3 mm, vias 1 -> 0
- net Net-(D18-A): track 12.5 -> 20.2 mm, vias 1 -> 2
- net Net-(D10-A): track 12.5 -> 20.1 mm, vias 1 -> 0
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
Commit message: routing cleanup
freerouting moment
Routing:
- net /Col2: track 224.9 -> 158.2 mm, vias 4 -> 6
- net /Col4: track 261.2 -> 204.1 mm, vias 3 -> 4
- net /Col5: track 182.1 -> 142.0 mm, vias 9 -> 10
- net Net-(D2-A): track 50.3 -> 18.6 mm, vias 1 -> 2
- net Net-(D4-A): track 34.7 -> 14.3 mm, vias 0 -> 1
- net /Row1: track 179.6 -> 160.1 mm, vias 0 -> 1
- net /Col3: track 187.1 -> 177.6 mm
- net Net-(D18-A): track 20.2 -> 11.3 mm, vias 2 -> 1
- net Net-(D3-A): track 17.7 -> 11.4 mm, vias 2 -> 1
- net Net-(D13-A): track 17.0 -> 11.1 mm
- net Net-(D1-A): track 28.1 -> 23.2 mm, vias 1 -> 0
- net /Col6: track 144.3 -> 140.4 mm
- net Net-(D5-A): track 15.5 -> 12.4 mm
- net Net-(D8-A): track 22.5 -> 19.9 mm, vias 2 -> 0
- net +3V3: track 33.2 -> 35.7 mm, vias 5 -> 1
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
Commit message: outline svg
Other:
- board outline added: 143.8 x 121.2 mm
Changed lines of the file:
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@@
 			(psnegative no)
 			(psa4output no)
-			(plot_black_and_white yes)
+			(plot_black_and_white no)
 			(sketchpadsonfab no)
 			(plotpadnumbers no)
@@
 		(embedded_fonts no)
 	)
+	(gr_poly
+		(pts
+			(xy 156.707505 31.155508) (xy 169.280487 31.727008) (xy 179.186493 37.823009) (xy 211.380997 38.20401)
+			(xy 211 120.5) (xy 184.711014 141.455017) (xy 173.662003 144.693511) (xy 149.278016 144.503005) (xy 142.801011 137.454513)
+			(xy 142.991501 121.833511) (xy 127.751503 106.97451) (xy 120.321999 106.403007) (xy 114.416504 110.975013)
+			(xy 79.745499 110.594009) (xy 67.553505 98.973503) (xy 67.743996 53.825012) (xy 73.459 47.919509)
+			(xy 88.127503 46.205009) (xy 92.509003 40.299507) (xy 105.653496 38.775508) (xy 109.654007 31.53651)
+			(xy 129.275498 31.155508) (xy 135.371506 23.535509) (xy 150.992508 23.535509)
+		)
+		(stroke
+			(width 0.762)
+			(type solid)
+		)
+		(fill no)
+		(layer "Edge.Cuts")
+	)
 	(segment
 		(start 125.4425 51.5007)
@@
 		(net 47)
 	)
+	(group ""
+		(members "5660904b-f26e-4944-8cb8-066b74f2d2e6")
+	)
 	(embedded_fonts no)
