File: kicad_nrf52840/V3.kicad_pcb (KiCad board)
At the start: 2 copper layers, 150.9 x 130.2 mm, 47 parts, among them SW1 KS33_SW_HS, SW10 KS33_SW_HS, SW11 KS33_SW_HS, SW12 KS33_SW_HS, SW13 KS33_SW_HS, SW14 KS33_SW_HS, SW15 KS33_SW_HS, SW16 KS33_SW_HS, SW17 KS33_SW_HS, SW18 KS33_SW_HS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

Commit message: update
Parts:
- SW1, SW10, SW11, SW12, SW13, SW14, SW15, SW16, SW17, SW18, SW19, SW2, SW20, SW21, SW22, SW3, SW4, SW5, SW6, SW7, SW8, SW9: footprint keyswitches:Kailh_socket_MX_reversible -> keyswitches:Kailh_socket_PG1350_reversible
Connections:
- U1 pad 18: unconnected-(U1-P0.29-LF-Pad18) -> /Col6
- U1 pad 19: unconnected-(U1-P0.02-LF-Pad19) -> /Col5
- U1 pad 20: unconnected-(U1-P1.15-LF-Pad20) -> /Col4
- U1 pad 25: /Col4 -> unconnected-(U1-P1.01-LF-Pad25)
- U1 pad 26: /Col5 -> unconnected-(U1-P1.02-LF-Pad26)
- U1 pad 27: /Col6 -> unconnected-(U1-P1.07-LF-Pad27)
Routing:
- net /Col4: track 163.9 -> 210.2 mm, vias 4 -> 5
- net /Col6: track 166.6 -> 151.8 mm, vias 4 -> 5
- net Net-(D19-A): track 12.2 -> 21.8 mm, vias 1 -> 0
- net Net-(D20-A): track 12.2 -> 21.6 mm, vias 1 -> 0
- net Net-(D6-A): track 12.2 -> 21.4 mm, vias 1 -> 0
- net Net-(D1-A): track 12.2 -> 21.4 mm, vias 1 -> 0
- net Net-(D12-A): track 12.2 -> 21.4 mm, vias 1 -> 0
- net Net-(D16-A): track 12.2 -> 21.4 mm, vias 1 -> 0
- net Net-(D10-A): track 12.2 -> 21.4 mm, vias 1 -> 0
- net Net-(D14-A): track 12.2 -> 21.4 mm, vias 1 -> 0
- net Net-(D4-A): track 12.2 -> 21.4 mm, vias 1 -> 0
- net Net-(D2-A): track 12.2 -> 21.4 mm, vias 1 -> 0
- net Net-(D8-A): track 12.2 -> 21.4 mm, vias 1 -> 0
- net Net-(D15-A): track 12.2 -> 21.3 mm, vias 1 -> 0
- net Net-(D9-A): track 12.2 -> 21.3 mm, vias 1 -> 0
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