File: kicad_nrf52840/V3.stretch_bkup.kicad_pcb (KiCad board)
At the start: 2 copper layers, 150.9 x 130.2 mm, 47 parts, among them SW1 KS33_SW_HS, SW10 KS33_SW_HS, SW11 KS33_SW_HS, SW12 KS33_SW_HS, SW13 KS33_SW_HS, SW14 KS33_SW_HS, SW15 KS33_SW_HS, SW16 KS33_SW_HS, SW17 KS33_SW_HS, SW18 KS33_SW_HS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

Commit message: nrf completed
Other:
- board outline removed
