File: kicad_nrf52840/V3.kicad_sch (KiCad schematic)
At the start: 47 parts, among them SW1 KS33_SW_HS, SW10 KS33_SW_HS, SW11 KS33_SW_HS, SW12 KS33_SW_HS, SW13 KS33_SW_HS, SW14 KS33_SW_HS, SW15 KS33_SW_HS, SW16 KS33_SW_HS, SW17 KS33_SW_HS, SW18 KS33_SW_HS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

Commit message: routing
Connections:
- net +3V3: now also U1.16 (3V3)
- net Col1: now also SW13.1, SW18.1, SW7.1; no longer SW15.1, SW4.1, SW9.1
- net Col2: now also SW11.1, SW17.1; no longer SW10.1, SW16.1
- net Col3: now also SW15.1, SW19.1, SW3.1, SW9.1; no longer SW1.1, SW13.1, SW2.1, SW7.1
- net Col4: now also SW1.1, SW12.1, SW6.1; no longer SW14.1, SW3.1, SW8.1
- net Col5: now also SW14.1, SW2.1, SW8.1; no longer SW12.1, SW18.1, SW6.1
- net Col6: now also SW10.1, SW16.1, SW4.1; no longer SW11.1, SW17.1, SW19.1
- net Row1: now also D1.1 (K), D2.1 (K), D3.1 (K), D7.1 (K)
- net Row2: now also D11.1 (K), D13.1 (K), D6.1 (K); no longer D12.1 (K), D17.1 (K), D7.1 (K)
- net Row3: now also D12.1 (K), D17.1 (K); no longer D13.1 (K), D19.1 (K)
- net Row4: now also D19.1 (K); no longer D1.1 (K)
Other:
- moved on the sheet: D1, D10, D11, D12, D13, D14, D15, D16, D17, D18, D19, D2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

Commit message: full routing
Connections:
- net Col1: now also U1.10 (P0.11); no longer U1.26 (P1.02-LF)
- net Col2: now also U1.9 (P1.00); no longer U1.27 (P1.07-LF)
Changed lines of the file:
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@@
+	(wire
+		(pts
+			(xy 186.69 60.96) (xy 191.77 60.96)
+		)
+		(stroke
+			(width 0)
+			(type default)
+		)
+	)
+	(wire
+		(pts
+			(xy 186.69 58.42) (xy 191.77 58.42)
+		)
+		(stroke
+			(width 0)
+			(type default)
+		)
+	)
 	(wire
 		(pts
@@
 	)
 	(label "Col2"
-		(at 210.82 76.2 90)
+		(at 186.69 58.42 0)
 		(effects
 			(font
@@
 	)
 	(label "Col1"
-		(at 208.28 76.2 90)
+		(at 186.69 60.96 0)
 		(effects
 			(font

Commit message: nrf completed
Parts:
- added SW23: Slide_Switch_SPDT_P3mm_10x5x10mm, PCM_SL_Devices:Slide_Switch_SPDT_P3mm_10x5x10mm, symbol PCM_SL_Devices:Slide_Switch_SPDT_P3mm_10x5x10mm
Connections:
- net B+: now also SW23.3; no longer BT1.1 (+)
- net Col2: now also U1.11 (P1.04-LF); no longer U1.9 (P1.00)
- net Col3: now also U1.12 (P1.06-LF); no longer U1.24 (P0.09-LF)
- net Col4: now also U1.25 (P1.01-LF); no longer U1.23 (P0.10-LF)
- net Col5: now also U1.26 (P1.02-LF); no longer U1.22 (P1.11-LF)
- net Col6: now also U1.27 (P1.07-LF); no longer U1.21 (P1.13-LF)
- net Row1: now also U1.24 (P0.09-LF); no longer U1.20 (P1.15-LF)
- net Row2: now also U1.23 (P0.10-LF); no longer U1.19 (P0.02-LF)
- net Row3: now also U1.22 (P1.11-LF); no longer U1.18 (P0.29-LF)
- net Row4: now also U1.21 (P1.13-LF); no longer U1.17 (P0.31-LF)
- net SCL: now also U1.6 (P0.20); no longer U1.12 (P1.06-LF)
- net SDA: now also U1.5 (P0.17); no longer U1.11 (P1.04-LF)
- new net: BT1.1 (+), SW23.1

Commit message: update
Parts:
- SW1, SW10, SW11, SW12, SW13, SW14, SW15, SW16, SW17, SW18, SW19, SW2, SW20, SW21, SW22, SW3, SW4, SW5, SW6, SW7, SW8, SW9: footprint keyswitches:Kailh_socket_MX_reversible -> keyswitches:Kailh_socket_PG1350_reversible
Connections:
- net Col4: now also U1.20 (P1.15-LF); no longer U1.25 (P1.01-LF)
- net Col5: now also U1.19 (P0.02-LF); no longer U1.26 (P1.02-LF)
- net Col6: now also U1.18 (P0.29-LF); no longer U1.27 (P1.07-LF)
- no-connect marks 0 -> 1
Changed lines of the file:
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@@
 		(color 0 0 0 0)
 	)
+	(no_connect
+		(at 77.47 217.17)
+	)
 	(bus_entry
 		(at 200.66 20.32)
@@
 	(wire
 		(pts
+			(xy 234.95 50.8) (xy 229.87 50.8)
+		)
+		(stroke
+			(width 0)
+			(type default)
+		)
+	)
+	(wire
+		(pts
 			(xy 205.74 71.12) (xy 205.74 76.2)
 		)
@@
 	(wire
 		(pts
+			(xy 234.95 53.34) (xy 229.87 53.34)
+		)
+		(stroke
+			(width 0)
+			(type default)
+		)
+	)
+	(wire
+		(pts
 			(xy 110.49 33.02) (xy 110.49 49.53)
 		)
@@
 	(wire
 		(pts
+			(xy 234.95 55.88) (xy 229.87 55.88)
+		)
+		(stroke
+			(width 0)
+			(type default)
+		)
+	)
+	(wire
+		(pts
 			(xy 115.57 81.28) (xy 128.27 81.28)
 		)
@@
 	)
 	(label "Col6"
-		(at 210.82 76.2 90)
+		(at 234.95 50.8 180)
 		(effects
 			(font
 				(size 1.27 1.27)
 			)
-			(justify left bottom)
+			(justify right bottom)
 		)
 	)
 	(label "Col4"
-		(at 205.74 76.2 90)
+		(at 234.95 55.88 180)
 		(effects
 			(font
 				(size 1.27 1.27)
 			)
-			(justify left bottom)
+			(justify right bottom)
 		)
 	)
@@
 	)
 	(label "Col5"
-		(at 208.28 76.2 90)
+		(at 234.95 53.34 180)
 		(effects
 			(font
 				(size 1.27 1.27)
 			)
-			(justify left bottom)
+			(justify right bottom)
 		)
 	)
@@
 			)
 		)
-		(property "Footprint" "keyswitches:Kailh_socket_MX_reversible"
+		(property "Footprint" "keyswitches:Kailh_socket_PG1350_reversible"
 			(at 113.03 90.17 0)
 			(effects
@@
 			)
 		)
-		(property "Footprint" "keyswitches:Kailh_socket_MX_reversible"
+		(property "Footprint" "keyswitches:Kailh_socket_PG1350_reversible"
 			(at 100.33 71.12 0)
 			(effects
@@
 			)
 		)
-		(property "Footprint" "keyswitches:Kailh_socket_MX_reversible"
+		(property "Footprint" "keyswitches:Kailh_socket_PG1350_reversible"
 			(at 113.03 71.12 0)
 			(effects
@@
 			)
 		)
-		(property "Footprint" "keyswitches:Kailh_socket_MX_reversible"
+		(property "Footprint" "keyswitches:Kailh_socket_PG1350_reversible"
 			(at 74.93 71.12 0)
 			(effects
@@
 			)
 		)
-		(property "Footprint" "keyswitches:Kailh_socket_MX_reversible"
+		(property "Footprint" "keyswitches:Kailh_socket_PG1350_reversible"
 			(at 125.73 71.12 0)
 			(effects
@@
 			)
 		)
-		(property "Footprint" "keyswitches:Kailh_socket_MX_reversible"
+		(property "Footprint" "keyswitches:Kailh_socket_PG1350_reversible"
 			(at 87.63 35.56 0)
 			(effects
@@
 			)
 		)
-		(property "Footprint" "keyswitches:Kailh_socket_MX_reversible"
+		(property "Footprint" "keyswitches:Kailh_socket_PG1350_reversible"
 			(at 125.73 35.56 0)
 			(effects
@@
 			)
 		)
-		(property "Footprint" "keyswitches:Kailh_socket_MX_reversible"
+		(property "Footprint" "keyswitches:Kailh_socket_PG1350_reversible"
 			(at 138.43 52.07 0)
 			(effects
@@
 			)
 		)
-		(property "Footprint" "keyswitches:Kailh_socket_MX_reversible"
+		(property "Footprint" "keyswitches:Kailh_socket_PG1350_reversible"
 			(at 87.63 52.07 0)
 			(effects
@@
 			)
 		)
-		(property "Footprint" "keyswitches:Kailh_socket_MX_reversible"
+		(property "Footprint" "keyswitches:Kailh_socket_PG1350_reversible"
 			(at 113.03 35.56 0)
 			(effects
@@
 			)
 		)
-		(property "Footprint" "keyswitches:Kailh_socket_MX_reversible"
+		(property "Footprint" "keyswitches:Kailh_socket_PG1350_reversible"
 			(at 125.73 90.17 0)
 			(effects
@@
 			)
 		)
-		(property "Footprint" "keyswitches:Kailh_socket_MX_reversible"
+		(property "Footprint" "keyswitches:Kailh_socket_PG1350_reversible"
 			(at 74.93 35.56 0)
 			(effects
@@
 			)
 		)
-		(property "Footprint" "keyswitches:Kailh_socket_MX_reversible"
+		(property "Footprint" "keyswitches:Kailh_socket_PG1350_reversible"
 			(at 138.43 71.12 0)
 			(effects
@@
 			)
 		)
-		(property "Footprint" "keyswitches:Kailh_socket_MX_reversible"
+		(property "Footprint" "keyswitches:Kailh_socket_PG1350_reversible"
 			(at 138.43 35.56 0)
 			(effects
@@
 			)
 		)
-		(property "Footprint" "keyswitches:Kailh_socket_MX_reversible"
+		(property "Footprint" "keyswitches:Kailh_socket_PG1350_reversible"
 			(at 100.33 90.17 0)
 			(effects
@@
 			)
 		)
-		(property "Footprint" "keyswitches:Kailh_socket_MX_reversible"
+		(property "Footprint" "keyswitches:Kailh_socket_PG1350_reversible"
 			(at 125.73 52.07 0)
 			(effects
@@
 			)
 		)
-		(property "Footprint" "keyswitches:Kailh_socket_MX_reversible"
+		(property "Footprint" "keyswitches:Kailh_socket_PG1350_reversible"
 			(at 100.33 52.07 0)
 			(effects
@@
 			)
 		)
-		(property "Footprint" "keyswitches:Kailh_socket_MX_reversible"
+		(property "Footprint" "keyswitches:Kailh_socket_PG1350_reversible"
 			(at 138.43 90.17 0)
 			(effects
@@
 			)
 		)
-		(property "Footprint" "keyswitches:Kailh_socket_MX_reversible"
+		(property "Footprint" "keyswitches:Kailh_socket_PG1350_reversible"
 			(at 87.63 71.12 0)
 			(effects
@@
 			)
 		)
-		(property "Footprint" "keyswitches:Kailh_socket_MX_reversible"
+		(property "Footprint" "keyswitches:Kailh_socket_PG1350_reversible"
 			(at 100.33 35.56 0)
 			(effects
@@
 			)
 		)
-		(property "Footprint" "keyswitches:Kailh_socket_MX_reversible"
+		(property "Footprint" "keyswitches:Kailh_socket_PG1350_reversible"
 			(at 113.03 52.07 0)
 			(effects
@@
 			)
 		)
-		(property "Footprint" "keyswitches:Kailh_socket_MX_reversible"
+		(property "Footprint" "keyswitches:Kailh_socket_PG1350_reversible"
 			(at 74.93 52.07 0)
 			(effects
