File: kicad_v4/esp32_s3_port.kicad_pcb (KiCad board)
At the start: 2 copper layers, 144.8 x 108.6 mm, 45 parts, among them J1 AudioJack4, J2 AudioJack4, SW1 KS33_SW_HS, SW10 KS33_SW_HS, SW11 KS33_SW_HS, SW12 KS33_SW_HS, SW13 KS33_SW_HS, SW14 KS33_SW_HS, SW15 KS33_SW_HS, SW16 KS33_SW_HS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

Commit message: signature
Routing:
- net GND: track 40.8 -> 17.4 mm, vias 8 -> 16
